Commit message: version 1.0.3

File: urdf/Final_Assembly2.xacro (robot description, xacro)
@@ -24,5 +24,5 @@
       <origin xyz="0 0 ${ofset_z}" rpy="0 0 0" />
       <geometry>
-        <mesh filename="package://lidar_hokuyo/meshes/base_link.STL" />
+        <mesh filename="package://robot_hokuyo/meshes/base_link.STL" />
       </geometry>
       <material name="">
@@ -33,5 +33,5 @@
       <origin xyz="0 0 ${ofset_z}" rpy="0 0 0" />
       <geometry>
-        <mesh filename="package://lidar_hokuyo/meshes/base_link.STL" />
+        <mesh filename="package://robot_hokuyo/meshes/base_link.STL" />
       </geometry>
     </collision>
@@ -63,5 +63,5 @@
       <origin xyz="0 0 0" rpy="0 0 0" />
       <geometry>
-        <mesh filename="package://lidar_hokuyo/meshes/right_wheel.STL" />
+        <mesh filename="package://robot_hokuyo/meshes/right_wheel.STL" />
       </geometry>
       <material name="">
@@ -72,5 +72,5 @@
       <origin xyz="0 0 0" rpy="0 0 0" />
       <geometry>
-        <mesh filename="package://lidar_hokuyo/meshes/right_wheel.STL" />
+        <mesh filename="package://robot_hokuyo/meshes/right_wheel.STL" />
       </geometry>
     </collision>
@@ -103,5 +103,5 @@
       <origin xyz="0 0 0" rpy="0 0 0" />
       <geometry>
-        <mesh filename="package://lidar_hokuyo/meshes/left_wheel.STL" />
+        <mesh filename="package://robot_hokuyo/meshes/left_wheel.STL" />
       </geometry>
       <material name="">
@@ -112,5 +112,5 @@
       <origin xyz="0 0 0" rpy="0 0 0" />
       <geometry>
-        <mesh filename="package://lidar_hokuyo/meshes/left_wheel.STL" />
+        <mesh filename="package://robot_hokuyo/meshes/left_wheel.STL" />
       </geometry>
     </collision>
@@ -143,5 +143,5 @@
       <origin xyz="0 0 0" rpy="0 0 0" />
       <geometry>
-        <mesh filename="package://lidar_hokuyo/meshes/front_caster.STL" />
+        <mesh filename="package://robot_hokuyo/meshes/front_caster.STL" />
       </geometry>
       <material name="">
@@ -152,5 +152,5 @@
       <origin xyz="0 0 0" rpy="0 0 0" />
       <geometry>
-        <mesh filename="package://lidar_hokuyo/meshes/front_caster.STL" />
+        <mesh filename="package://robot_hokuyo/meshes/front_caster.STL" />
       </geometry>
     </collision>
@@ -183,5 +183,5 @@
       <origin xyz="0 0 0" rpy="0 0 0" />
       <geometry>
-        <mesh filename="package://lidar_hokuyo/meshes/back_caster.STL" />
+        <mesh filename="package://robot_hokuyo/meshes/back_caster.STL" />
       </geometry>
       <material name="">
@@ -192,5 +192,5 @@
       <origin xyz="0 0 0" rpy="0 0 0" />
       <geometry>
-        <mesh filename="package://lidar_hokuyo/meshes/back_caster.STL" />
+        <mesh filename="package://robot_hokuyo/meshes/back_caster.STL" />
       </geometry>
     </collision>
@@ -223,5 +223,5 @@
       <origin xyz="0 0 0" rpy="0 0 0" />
       <geometry>
-        <mesh filename="package://lidar_hokuyo/meshes/laser_link.STL" />
+        <mesh filename="package://robot_hokuyo/meshes/laser_link.STL" />
       </geometry>
       <material name="">
@@ -234,5 +234,5 @@
         rpy="0 0 0" />
       <geometry>
-        <mesh filename="package://lidar_hokuyo/meshes/laser_link.STL" />
+        <mesh filename="package://robot_hokuyo/meshes/laser_link.STL" />
       </geometry>
     </collision>

Commit message: verrsion 1.0.4

File: urdf/Final_Assembly2.xacro (robot description, xacro)
@@ -30,10 +30,4 @@
       </material>
     </visual>
-    <collision>
-      <origin xyz="0 0 ${ofset_z}" rpy="0 0 0" />
-      <geometry>
-        <mesh filename="package://robot_hokuyo/meshes/base_link.STL" />
-      </geometry>
-    </collision>
   </link>
   <joint name="base_link_joint" type="fixed">
@@ -69,10 +63,4 @@
       </material>
     </visual>
-    <collision>
-      <origin xyz="0 0 0" rpy="0 0 0" />
-      <geometry>
-        <mesh filename="package://robot_hokuyo/meshes/right_wheel.STL" />
-      </geometry>
-    </collision>
   </link>
   <joint name="right_joint" type="continuous">
@@ -109,10 +97,4 @@
       </material>
     </visual>
-    <collision>
-      <origin xyz="0 0 0" rpy="0 0 0" />
-      <geometry>
-        <mesh filename="package://robot_hokuyo/meshes/left_wheel.STL" />
-      </geometry>
-    </collision>
   </link>
   <joint name="left_joint" type="continuous">
@@ -149,10 +131,4 @@
       </material>
     </visual>
-    <collision>
-      <origin xyz="0 0 0" rpy="0 0 0" />
-      <geometry>
-        <mesh filename="package://robot_hokuyo/meshes/front_caster.STL" />
-      </geometry>
-    </collision>
   </link>
   <joint name="front_joint" type="fixed">
@@ -189,10 +165,4 @@
       </material>
     </visual>
-    <collision>
-      <origin xyz="0 0 0" rpy="0 0 0" />
-      <geometry>
-        <mesh filename="package://robot_hokuyo/meshes/back_caster.STL" />
-      </geometry>
-    </collision>
   </link>
   <joint name="back_joint" type="fixed">
@@ -229,12 +199,4 @@
       </material>
     </visual>
-    <collision>
-      <origin
-        xyz="0 0 0"
-        rpy="0 0 0" />
-      <geometry>
-        <mesh filename="package://robot_hokuyo/meshes/laser_link.STL" />
-      </geometry>
-    </collision>
   </link>
   <joint name="lidar_joint" type="fixed">

Commit message: meger camera to package

File: urdf/Final_Assembly2.xacro (robot description, xacro)
@@ -206,4 +206,24 @@
     <parent link="base_link" />
     <child link="lidar_link" />
+    <axis xyz="0 0 0" />
+  </joint>
+  <!-- ######################### camera_link ######################### -->
+  <link name="camera_link">
+    <visual>
+      <origin xyz="0 0 0" rpy="0 0 0" />
+      <geometry>
+        <box size="0.030 0.10 0.035"/>
+      </geometry>
+      <material name="">
+        <color rgba="0.701960784313725 0.552941176470588 0.00392156862745098 1" />
+      </material>
+    </visual>
+  </link>
+  <joint name="camera_joint" type="fixed">
+    <origin
+      xyz="0.022 0 ${ofset_z + 0.30}"
+      rpy="0 0 0" />
+    <parent link="base_link" />
+    <child link="camera_link" />
     <axis xyz="0 0 0" />
   </joint>
@@ -225,6 +245,6 @@
       <publish_wheel_tf>true</publish_wheel_tf>
       <command_topic>cmd_vel</command_topic>
-      <odometry_topic>odom</odometry_topic>
-      <odometry_frame>odom</odometry_frame>
+      <odometry_topic>wheel_odom</odometry_topic>
+      <odometry_frame>wheel_odom</odometry_frame>
       <robot_base_frame>base_footprint</robot_base_frame>
     </plugin>

Commit message: fixed xacro

File: urdf/Final_Assembly2.xacro (robot description, xacro)
@@ -24,5 +24,6 @@
       <origin xyz="0 0 ${ofset_z}" rpy="0 0 0" />
       <geometry>
-        <mesh filename="package://robot_hokuyo/meshes/base_link.STL" />
+        <box size="0.20 0.18 0.06"/>
+        <!-- <mesh filename="package://robot_hokuyo/meshes/base_link.STL" /> -->
       </geometry>
       <material name="">
@@ -57,5 +58,6 @@
       <origin xyz="0 0 0" rpy="0 0 0" />
       <geometry>
-        <mesh filename="package://robot_hokuyo/meshes/right_wheel.STL" />
+        <cylinder radius="0.0325" length="0.02"/>
+        <!-- <mesh filename="package://robot_hokuyo/meshes/right_wheel.STL" /> -->
       </geometry>
       <material name="">
@@ -91,5 +93,6 @@
       <origin xyz="0 0 0" rpy="0 0 0" />
       <geometry>
-        <mesh filename="package://robot_hokuyo/meshes/left_wheel.STL" />
+        <cylinder radius="0.0325" length="0.02"/>
+        <!-- <mesh filename="package://robot_hokuyo/meshes/left_wheel.STL" /> -->
       </geometry>
       <material name="">
@@ -125,5 +128,6 @@
       <origin xyz="0 0 0" rpy="0 0 0" />
       <geometry>
-        <mesh filename="package://robot_hokuyo/meshes/front_caster.STL" />
+        <sphere radius="0.015"/>
+        <!-- <mesh filename="package://robot_hokuyo/meshes/front_caster.STL" /> -->
       </geometry>
       <material name="">
@@ -159,5 +163,6 @@
       <origin xyz="0 0 0" rpy="0 0 0" />
       <geometry>
-        <mesh filename="package://robot_hokuyo/meshes/back_caster.STL" />
+        <sphere radius="0.015"/>
+        <!-- <mesh filename="package://robot_hokuyo/meshes/back_caster.STL" /> -->
       </geometry>
       <material name="">
@@ -193,5 +198,6 @@
       <origin xyz="0 0 0" rpy="0 0 0" />
       <geometry>
-        <mesh filename="package://robot_hokuyo/meshes/laser_link.STL" />
+        <cylinder radius="0.035" length="0.05"/>
+        <!-- <mesh filename="package://robot_hokuyo/meshes/laser_link.STL" /> -->
       </geometry>
       <material name="">
@@ -236,5 +242,5 @@
       <!-- kinematics -->
       <wheel_separation>0.236</wheel_separation>
-      <wheel_diameter>0.13</wheel_diameter>
+      <wheel_diameter>0.065</wheel_diameter>
       <!-- limits -->
       <max_wheel_torque>80</max_wheel_torque>

Commit message: fixed xacro

File: urdf/Final_Assembly2.xacro (robot description, xacro)
@@ -24,5 +24,5 @@
       <origin xyz="0 0 ${ofset_z}" rpy="0 0 0" />
       <geometry>
-        <box size="0.20 0.18 0.06"/>
+        <cylinder radius="0.1" length="0.005"/>
         <!-- <mesh filename="package://robot_hokuyo/meshes/base_link.STL" /> -->
       </geometry>
@@ -56,7 +56,7 @@
     </inertial>
     <visual>
-      <origin xyz="0 0 0" rpy="0 0 0" />
-      <geometry>
-        <cylinder radius="0.0325" length="0.02"/>
+      <origin xyz="0 0 0" rpy="1.5708 0 0" />
+      <geometry>
+        <cylinder radius="0.0325" length="0.026"/>
         <!-- <mesh filename="package://robot_hokuyo/meshes/right_wheel.STL" /> -->
       </geometry>
@@ -91,7 +91,7 @@
     </inertial>
     <visual>
-      <origin xyz="0 0 0" rpy="0 0 0" />
-      <geometry>
-        <cylinder radius="0.0325" length="0.02"/>
+      <origin xyz="0 0 0" rpy="1.5708 0 0" />
+      <geometry>
+        <cylinder radius="0.0325" length="0.026"/>
         <!-- <mesh filename="package://robot_hokuyo/meshes/left_wheel.STL" /> -->
       </geometry>
